File: truck_drivers.kicad_sch (KiCad schematic)
At the start: 44 parts

Commit message: add horn circuit
Parts:
- added D?: D, symbol Device:D
- added J?: TE_Faston_20-16AWG_Straight_Tab, TE_Faston_20-16AWG_Straight_Tab, symbol Toadly:TE_Faston_20-16AWG_Straight_Tab
- added Q?: ZXTN08400BFFCT, Package_TO_SOT_SMD:SOT-23, symbol Device:Q_NPN_BCE
- added R? (x2): 10k, symbol Device:R_US
Connections:
- net +12C: now also D?.1 (K)
- net GNDREF: now also Q?.3 (E), R?.2
- new net: Q?.1 (B), R?.1, R?.2
- new net: D?.2 (A), J?.1 (P1), J?.2 (P1), Q?.2 (C)
- new net HORN_EN: R?.1
Other:
- note added: "Horn"
- note added: "TODO: maybe pull this out, these should be individually controlled as they override high beams for flasher"
- note added: "TODO: probably want to individually control these for turn signalling?"
- note added: "To horn relay"
- moved on the sheet: C?, J?, R?, U?A, U?B, U?C

Commit message: add signal inputs
Other:
- note added: "TODO: isolate this"
- note added: "TODO: select diode, at least 200mA"
Changed lines of the file:
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@@
+    (effects (font (size 1.27 1.27)) (justify left bottom))
+  )
+  (text "TODO: select diode, at least 200mA" (at 166.37 135.89 0)
     (effects (font (size 1.27 1.27)) (justify left bottom))
   )
@@
     (effects (font (size 2 2)) (justify left bottom))
   )
+  (text "TODO: isolate this" (at 149.86 158.75 0)
+    (effects (font (size 1.27 1.27)) (justify left bottom))
+  )
   (text "To horn relay" (at 227.33 135.89 0)

Commit message: select 1n4148w for horn flywheel diode
Parts:
- removed D?: D, symbol Device:D
- added D?: 1N4148W, Diode_SMD:D_SOD-123, symbol Diode:1N4148W
Connections:
- net +12C: now also D?.1 (K)
- net at J?.1 (P1), J?.2 (P1), Q?.2 (C): now also D?.2 (A)
Other:
- note removed: "TODO: select diode, at least 200mA"
Changed lines of the file:
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@@
-    (effects (font (size 1.27 1.27)) (justify left bottom))
-  )
-  (text "TODO: select diode, at least 200mA" (at 166.37 135.89 0)
     (effects (font (size 1.27 1.27)) (justify left bottom))
   )
@@
     (pin "2")
   )
-  (symbol (lib_id "Device:D") (at 205.74 138.43 0) (unit 1)
-    (in_bom yes) (on_board yes)
-    (property "Reference" "D?" (id 0) (at 205.74 133.35 0))
-    (property "Value" "D" (id 1) (at 205.74 135.89 0))
-    (property "Footprint" "" (id 2) (at 205.74 138.43 0)
-      (effects (font (size 1.27 1.27)) hide)
-    )
-    (property "Datasheet" "~" (id 3) (at 205.74 138.43 0)
-      (effects (font (size 1.27 1.27)) hide)
-    )
-    (pin "1")
-    (pin "2")
-  )
   (symbol (lib_id "Toadly:VND5160J") (at 95.25 139.7 0) (unit 2)
     (in_bom yes) (on_board yes) (fields_autoplaced)
@@
     (pin "1")
   )
+  (symbol (lib_id "Diode:1N4148W") (at 205.74 138.43 0) (unit 1)
+    (in_bom yes) (on_board yes) (fields_autoplaced)
+    (property "Reference" "D?" (id 0) (at 205.74 132.08 0))
+    (property "Value" "1N4148W" (id 1) (at 205.74 134.62 0))
+    (property "Footprint" "Diode_SMD:D_SOD-123" (id 2) (at 205.74 142.875 0)
+      (effects (font (size 1.27 1.27)) hide)
+    )
+    (property "Datasheet" "https://www.vishay.com/docs/85748/1n4148w.pdf" (id 3) (at 205.74 138.43 0)
+      (effects (font (size 1.27 1.27)) hide)
+    )
+    (pin "1")
+    (pin "2")
+  )
   (symbol (lib_id "Toadly:TE_Faston_20-16AWG_Straight_Tab") (at 116.84 50.8 0) (unit 1)

Commit message: annotate schematic
Parts:
- C10, C11, C12, C13, C14: renamed from C?; footprint (none) -> Capacitor_SMD:C_0805_2012Metric_Pad1.18x1.45mm_HandSolder
- R10, R11, R12, R13, R14, R15, R16, R17, R18, R19, R20, R21, R6, R7, R8, R9: renamed from R?; footprint (none) -> Resistor_SMD:R_0805_2012Metric_Pad1.20x1.40mm_HandSolder
- gave numbers to parts that had none: 18

Commit message: add compartment lights, switch to samd21j
Other:
- note added: "Side red lights above wheel wells"
- note added: "These are small lights above rear door and cab"
- note removed: "TODO: probably want to individually control these for turn signalling?"
Changed lines of the file:
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@@
     (effects (font (size 2 2)) (justify left bottom))
   )
-  (text "TODO: probably want to individually control\nthese for turn signalling?"
-    (at 172.72 63.5 0)
+  (text "These are small lights above rear\ndoor and cab" (at 177.8 24.13 0)
     (effects (font (size 1.27 1.27)) (justify left bottom))
   )
@@
     (effects (font (size 1.27 1.27)) (justify left bottom))
   )
-  (text "Intersection Lights" (at 24.13 142.24 0)
+  (text "Intersection Lights" (at 20.32 139.7 0)
     (effects (font (size 2 2)) (justify left bottom))
   )
@@
     (effects (font (size 2 2)) (justify left bottom))
   )
+  (text "Side red lights above wheel wells" (at 20.32 143.51 0)
+    (effects (font (size 1.27 1.27)) (justify left bottom))
+  )
   (text "Chime + Backup Alarm" (at 24.13 25.4 0)
