File: signals.kicad_sch (KiCad schematic)
At the start: 134 parts, among them J12 TE_Faston_20-16AWG_Straight_T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, J13 TE_Faston_20-16AWG_Straight_T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, J14 TE_Faston_20-16AWG_Straight_T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, J15 TE_Faston_20-16AWG_Straight_T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, J16 TE_Faston_20-16AWG_Straight_T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, J17 TE_Faston_20-16AWG_Straight_T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, J18 TE_Faston_20-16AWG_Straight_T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, J19 TE_Faston_20-16AWG_Straight_T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, J20 TE_Faston_20-16AWG_Straight_T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, J21 TE_Faston_20-16AWG_Straight_T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

Commit message: route sense input tracks
Connections:
- net CAB_1_SENSE: now also U5.9; no longer U5.15
- net CAB_2_SENSE: now also U5.11; no longer U5.13
- net CAB_3_SENSE: now also U5.13; no longer U5.11
- net CAB_4_SENSE: now also U5.15; no longer U5.9
- net at R34.1, R36.1: now also U5.3; no longer U5.5
- net at J23.1 (P1), J23.2 (P1): now also R75.2; no longer R54.2
- net at J26.1 (P1), J26.2 (P1): now also R80.2; no longer R79.2
- net at R33.1, R35.1: now also U5.1; no longer U5.7
- net at J15.1 (P1), J15.2 (P1): now also R9.1; no longer R12.1
- net at J12.1 (P1), J12.2 (P1): now also R10.1; no longer R9.1
- net at J25.1 (P1), J25.2 (P1): now also R53.2; no longer R76.2
- net at J19.1 (P1), J19.2 (P1): now also R31.1; no longer R32.1
- net at R14.1, R16.1: now also U5.7; no longer U5.1
- net at J22.1 (P1), J22.2 (P1): now also R76.2; no longer R51.2
- net at J13.1 (P1), J13.2 (P1): now also R11.1; no longer R10.1
- net at J21.1 (P1), J21.2 (P1): now also R51.2; no longer R53.2
- net at J16.1 (P1), J16.2 (P1): now also R32.1; no longer R29.1
- net at J24.1 (P1), J24.2 (P1): now also R52.2; no longer R75.2
- net at J27.1 (P1), J27.2 (P1): now also R79.2; no longer R80.2
- net at J14.1 (P1), J14.2 (P1): now also R12.1; no longer R11.1
- net at J20.1 (P1), J20.2 (P1): now also R54.2; no longer R52.2
- net at J18.1 (P1), J18.2 (P1): now also R30.1; no longer R31.1
- net at J17.1 (P1), J17.2 (P1): now also R29.1; no longer R30.1
- net at R13.1, R15.1: now also U5.5; no longer U5.3
Other:
- moved on the sheet: J12, J13, J14, J15, J16, J17, J18, J19, J20, J21, J22, J23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
